Commit message: backup

File: src/udacity_bot/urdf/udacity_bot.xacro (robot description, xacro)
@@ -67,5 +67,5 @@
     </collision>
     <visual name='front_caster_visual'>
-      <origin xyz="0.15 0 -0.05" rpy=" 0 0 0"/>
+      <origin xyz="0.15 0.0 -0.05" rpy=" 0 0 0"/>
       <geometry>
         <sphere radius="0.05"/>
@@ -75,16 +75,16 @@
   <link name="left_wheel">
     <inertial>
-      <origin xyz="0 0 0" rpy="0 1.5707 1.5707" />
-      <mass value="5"/>
+      <origin xyz="0.0 0.0 0.0" rpy="0.0 1.5707 1.5707" />
+      <mass value="5.0"/>
       <inertia ixx="0.1" ixy="0" ixz="0" iyy="0.1" iyz="0" izz="0.1" />
     </inertial>
     <collision name='collision'>
-      <origin xyz="0 0 0" rpy=" 0 1.5707 1.5707"/>
+      <origin xyz="0.0 0.0 0.0" rpy=" 0 1.5707 1.5707"/>
       <geometry>
         <cylinder radius="0.1" length="0.05"/>
       </geometry>
     </collision>
-    <visual>
-      <origin xyz="0 0 0" rpy="0 1.5707 1.5707" />
+    <visual name="lef_wheel_visual">
+      <origin xyz="0.0 0.0 0.0" rpy="0 1.5707 1.5707" />
       <geometry>
         <cylinder radius="0.1" length="0.05"/>
@@ -93,5 +93,5 @@
   </link>
   <joint type="continuous" name="left_wheel_hinge">
-    <origin xyz="0 0.15 0" rpy="0 0 0"/>
+    <origin xyz="0.0 0.15 0.0" rpy="0 0 0"/>
     <child link="left_wheel"/>
     <parent link="chassis"/>
@@ -102,16 +102,16 @@
   <link name="right_wheel">
     <inertial>
-      <origin xyz="0 0 0" rpy="0 1.5707 1.5707" />
-      <mass value="5"/>
+      <origin xyz="0.0 0.0 0.0" rpy="0.0 1.5707 1.5707" />
+      <mass value="5.0"/>
       <inertia ixx="0.1" ixy="0" ixz="0" iyy="0.1" iyz="0" izz="0.1" />
     </inertial>
     <collision name='collision'>
-      <origin xyz="0 0 0" rpy=" 0 1.5707 1.5707"/>
+      <origin xyz="0.0 0.0 0.0" rpy=" 0 1.5707 1.5707"/>
       <geometry>
         <cylinder radius="0.1" length="0.05"/>
       </geometry>
     </collision>
-    <visual>
-      <origin xyz="0 0 0" rpy="0 1.5707 1.5707" />
+    <visual name="right_wheel_visual">
+      <origin xyz="0.0 0.0 0.0" rpy="0 1.5707 1.5707" />
       <geometry>
         <cylinder radius="0.1" length="0.05"/>
@@ -120,5 +120,5 @@
   </link>
   <joint type="continuous" name="right_wheel_hinge">
-    <origin xyz="0 -0.15 0" rpy="0 0 0"/>
+    <origin xyz="0.0 -0.15 0.0" rpy="0 0 0"/>
     <child link="right_wheel"/>
     <parent link="chassis"/>

Commit message: feat: straight drive possible

File: src/udacity_bot/urdf/udacity_bot.xacro (robot description, xacro)
@@ -31,5 +31,5 @@
       <origin xyz="-0.15 0 -0.05" rpy=" 0 0 0"/>
       <geometry>
-        <sphere radius="0.05"/>
+        <sphere radius="0.045"/>
       </geometry>
       <surface>
@@ -38,6 +38,6 @@
             <mu>0</mu>
             <mu2>0</mu2>
-            <slip1>1.0</slip1>
-            <slip2>1.0</slip2>
+            <slip1>0.</slip1>
+            <slip2>0.</slip2>
           </ode>
         </friction>
@@ -53,5 +53,5 @@
       <origin xyz="0.15 0 -0.05" rpy=" 0 0 0"/>
       <geometry>
-        <sphere radius="0.05"/>
+        <sphere radius="0.045"/>
       </geometry>
       <surface>
@@ -60,6 +60,6 @@
             <mu>0</mu>
             <mu2>0</mu2>
-            <slip1>1.0</slip1>
-            <slip2>1.0</slip2>
+            <slip1>0.0</slip1>
+            <slip2>0.0</slip2>
           </ode>
         </friction>

Commit message: feat: wird besser

File: src/udacity_bot/urdf/udacity_bot.xacro (robot description, xacro)
@@ -36,6 +36,6 @@
         <friction>
           <ode>
-            <mu>0</mu>
-            <mu2>0</mu2>
+            <mu>0.1</mu>
+            <mu2>0.1</mu2>
             <slip1>0.</slip1>
             <slip2>0.</slip2>
@@ -58,6 +58,6 @@
         <friction>
           <ode>
-            <mu>0</mu>
-            <mu2>0</mu2>
+            <mu>0.1</mu>
+            <mu2>0.1</mu2>
             <slip1>0.0</slip1>
             <slip2>0.0</slip2>
@@ -155,5 +155,5 @@
 <!--LIDAR-->
 <link name="hokuyo">
-    <origin>0 0 0 0 0 0</origin>
+    <origin>0. 0 0 0 0 0</origin>
     <inertial>
       <origin xyz="0 0 0" rpy="0 0 0"/>
@@ -174,5 +174,5 @@
   </link>
   <joint type="fixed" name="hokuyo_joint">
-    <origin xyz="0.15 0 0.1" rpy="0 0 0"/>
+    <origin xyz="0.2 0 0.15" rpy="0 0 0"/>
     <child link="hokuyo" />
     <parent link="chassis" />
